File: sch_pcb/arduvga.kicad_pcb (KiCad board)
At the start: 2 copper layers, 69.6 x 54.4 mm, 11 parts, among them J1 Conn_01x04_Socket, J3 Conn_01x04_Socket, J5 DSUB15

Commit message: update pcb
Parts:
- moved R6 1.02 mm to (145.3, 104.1)
- moved J1 0.51 mm to (150.4, 117.9)
- moved J3 0.51 mm to (150.4, 108.7)
- moved R2 0.51 mm to (158.0, 93.5)
- moved R1 0.51 mm to (176.0, 78.7)
Routing:
- net Net-(A1-A3): track 39.3 -> 33.7 mm
- net Net-(J3-Pin_3): track 46.4 -> 41.6 mm
- net Net-(A1-A1): track 26.7 -> 22.0 mm
- net Net-(A1-A2): track 34.1 -> 31.4 mm
- net Net-(J5-Pad14): track 49.5 -> 47.1 mm
- net +5V: track 19.2 -> 18.6 mm
- net Net-(J5-Pad13): track 23.0 -> 23.5 mm

Commit message: update pcb
Parts:
- moved R4 0.51 mm to (163.6, 78.7)
Changed lines of the file:
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@@
   )
   (footprint "Resistor_THT:R_Axial_DIN0207_L6.3mm_D2.5mm_P7.62mm_Horizontal" (layer "F.Cu")
-    (at 163.068 78.74 180)
+    (at 163.576 78.74 180)
     (descr "Resistor, Axial_DIN0207 series, Axial, Horizontal, pin pitch=7.62mm, 0.25W = 1/4W, length*diameter=6.3*2.5mm^2, http://cdn-reichelt.de/documents/datenblatt/B400/1_4W%23YAG.pdf")
     (tags "Resistor Axial_DIN0207 series Axial Horizontal pin pitch 7.62mm 0.25W = 1/4W length 6.3mm diameter 2.5mm")
@@
   (segment (start 150.368 121.92) (end 150.368 117.856002) (width 1.25) (layer "B.Cu") (net 5))
   (segment (start 150.876 108.712) (end 151.892002 108.712) (width 1.25) (layer "B.Cu") (net 5))
-  (segment (start 169.094 96.964) (end 169.094 94.674) (width 1) (layer "B.Cu") (net 6))
-  (segment (start 169.164 92.314) (end 169.094 92.384) (width 0.5) (layer "B.Cu") (net 6))
-  (segment (start 169.094 92.384) (end 169.094 94.674) (width 1) (layer "B.Cu") (net 6))
-  (segment (start 167.114 102.689) (end 167.949 102.689) (width 0.75) (layer "B.Cu") (net 6))
-  (segment (start 167.949 102.689) (end 169.094 101.544) (width 0.75) (layer "B.Cu") (net 6))
-  (segment (start 149.86 115.316) (end 147.828 117.348) (width 1) (layer "B.Cu") (net 9))
-  (segment (start 165.608 121.92) (end 165.608 120.904) (width 1) (layer "B.Cu") (net 9))
-  (segment (start 160.02 115.316) (end 149.86 115.316) (width 1) (layer "B.Cu") (net 9))
-  (segment (start 165.608 120.904) (end 160.02 115.316) (width 1) (layer "B.Cu") (net 9))
+  (segment (start 169.094 96.964) (end 169.094 94.674) (width 1.25) (layer "B.Cu") (net 6))
+  (segment (start 169.164 92.314) (end 169.094 92.384) (width 1.25) (layer "B.Cu") (net 6))
+  (segment (start 169.094 92.384) (end 169.094 94.674) (width 1.25) (layer "B.Cu") (net 6))
+  (segment (start 167.114 102.689) (end 167.949 102.689) (width 1) (layer "B.Cu") (net 6))
+  (segment (start 167.949 102.689) (end 169.094 101.544) (width 1) (layer "B.Cu") (net 6))
+  (segment (start 147.828 116.332) (end 147.828 117.348) (width 1) (layer "B.Cu") (net 9))
+  (segment (start 159.004 115.316) (end 148.844 115.316) (width 1) (layer "B.Cu") (net 9))
+  (segment (start 165.608 121.92) (end 159.004 115.316) (width 1) (layer "B.Cu") (net 9))
+  (segment (start 148.844 115.316) (end 147.828 116.332) (width 1) (layer "B.Cu") (net 9))
   (segment (start 168.148 120.396) (end 161.036 113.284) (width 1) (layer "B.Cu") (net 10))
   (segment (start 168.148 121.92) (end 168.148 120.396) (width 1) (layer "B.Cu") (net 10))
@@
   (segment (start 173.228 119.888) (end 157.48 104.14) (width 1) (layer "B.Cu") (net 12))
   (segment (start 168.148 73.66) (end 168.148 78.486) (width 1.25) (layer "B.Cu") (net 17))
-  (segment (start 157.988 85.344) (end 157.988 84.074) (width 1) (layer "B.Cu") (net 19))
-  (segment (start 157.988 84.074) (end 160.528 81.534) (width 1) (layer "B.Cu") (net 19))
-  (segment (start 160.528 81.534) (end 160.528 73.66) (width 1) (layer "B.Cu") (net 19))
+  (segment (start 160.02 83.312) (end 160.02 74.168) (width 1) (layer "B.Cu") (net 19))
+  (segment (start 157.988 85.344) (end 160.02 83.312) (width 1) (layer "B.Cu") (net 19))
+  (segment (start 160.02 74.168) (end 160.528 73.66) (width 1) (layer "B.Cu") (net 19))
   (segment (start 157.988 73.66) (end 157.988 81.28) (width 1) (layer "B.Cu") (net 20))
   (segment (start 154.432 84.836) (end 154.432 87.884) (width 1) (layer "B.Cu") (net 20))
@@
   (segment (start 176.022 78.74) (end 176.022 96.774) (width 1) (layer "B.Cu") (net 36))
   (segment (start 177.8 77.216) (end 177.8 98.552) (width 1) (layer "B.Cu") (net 37))
+  (segment (start 163.576 78.74) (end 163.576 79.756) (width 1) (layer "B.Cu") (net 37))
+  (segment (start 169.418 81.28) (end 174.498 76.2) (width 1) (layer "B.Cu") (net 37))
+  (segment (start 177.8 98.552) (end 175.953 100.399) (width 1) (layer "B.Cu") (net 37))
   (segment (start 174.498 76.2) (end 176.784 76.2) (width 1) (layer "B.Cu") (net 37))
-  (segment (start 163.068 78.74) (end 165.608 81.28) (width 1) (layer "B.Cu") (net 37))
+  (segment (start 165.1 81.28) (end 169.418 81.28) (width 1) (layer "B.Cu") (net 37))
+  (segment (start 163.576 79.756) (end 165.1 81.28) (width 1) (layer "B.Cu") (net 37))
   (segment (start 175.953 100.399) (end 171.074 100.399) (width 1) (layer "B.Cu") (net 37))
   (segment (start 176.784 76.2) (end 177.8 77.216) (width 1) (layer "B.Cu") (net 37))
-  (segment (start 169.418 81.28) (end 174.498 76.2) (width 1) (layer "B.Cu") (net 37))
-  (segment (start 165.608 81.28) (end 169.418 81.28) (width 1) (layer "B.Cu") (net 37))
-  (segment (start 177.8 98.552) (end 175.953 100.399) (width 1) (layer "B.Cu") (net 37))
-  (segment (start 161.544 77.216) (end 161.544 90.424) (width 0.5) (layer "B.Cu") (net 39))
-  (segment (start 163.068 73.66) (end 163.068 75.692) (width 0.5) (layer "B.Cu") (net 39))
-  (segment (start 163.068 75.692) (end 161.544 77.216) (width 0.5) (layer "B.Cu") (net 39))
+  (segment (start 161.544 77.216) (end 161.544 90.424) (width 1) (layer "B.Cu") (net 39))
+  (segment (start 163.068 73.66) (end 163.068 75.692) (width 1) (layer "B.Cu") (net 39))
+  (segment (start 163.068 75.692) (end 161.544 77.216) (width 1) (layer "B.Cu") (net 39))
   (segment (start 161.609 98.109) (end 161.544 98.044) (width 1) (layer "B.Cu") (net 40))
   (segment (start 167.114 98.109) (end 161.609 98.109) (width 1) (layer "B.Cu") (net 40))
