File: sch_pcb/arduvga.kicad_pcb (KiCad board)
At the start: 2 copper layers, 69.6 x 54.4 mm, 11 parts, among them J1 Conn_01x04_Socket, J3 Conn_01x04_Socket, J5 DSUB15

Commit message: update pcb
Parts:
- moved R4 26.2 mm to (150.9, 101.6), turned to 90 degrees
- moved J5 6.17 mm to (173.3, 93.6)
- moved R6 0.51 mm to (145.3, 103.6)
Routing:
- net Net-(A1-D9): track 8.85 -> 20.5 mm
- net Net-(J5-Pad14): track 47.2 -> 38.3 mm
- net Net-(J5-Pad2): track 12.8 -> 19.5 mm
- net Net-(J5-Pad3): track 5.60 -> 11.9 mm
- net Net-(J5-Pad1): track 9.15 -> 15.4 mm
- net +5V: track 18.6 -> 24.9 mm
- net Net-(J3-Pin_3): track 41.6 -> 45.0 mm
- net Net-(A1-A3): track 33.7 -> 36.1 mm

Commit message: update pcb
Parts:
- A1: footprint Module:Arduino_UNO_R3 -> libs:Arduino_UNO_R3_OVAL
Routing:
- net Net-(A1-A2): track 31.4 -> 32.4 mm
- net Net-(A1-A1): track 22.0 -> 22.7 mm
