File: sch_pcb/arduvga.kicad_sch (KiCad schematic)
At the start: 17 parts, among them J1 Conn_01x04_Socket, J2 Conn_01x04_Pin, J3 Conn_01x04_Socket, J4 Conn_01x04_Pin, J5 DSUB15, SW1 Push, SW2 Push

Commit message: update sch
Other:
- note added: "R7: no se utiliza con los firmware "Arduino_VGA_Game.ino" y "VGAX_Bomber_v01.ino"."
Changed lines of the file:
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@@
+    (effects (font (size 1.27 1.27)) (justify left bottom))
+  )
+  (text "R7: no se utiliza con los firmware \"Arduino_VGA_Game.ino\" y \"VGAX_Bomber_v01.ino\"."
+    (at 53.34 130.81 0)
     (effects (font (size 1.27 1.27)) (justify left bottom))
   )

Commit message: update pcb
Parts:
- A1: footprint Module:Arduino_UNO_R3 -> libs:Arduino_UNO_R3_OVAL
Changed lines of the file:
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@@
       (effects (font (size 1.27 1.27)) (justify left))
     )
-    (property "Footprint" "Module:Arduino_UNO_R3" (at 113.03 83.82 0)
+    (property "Footprint" "libs:Arduino_UNO_R3_OVAL" (at 113.03 83.82 0)
       (effects (font (size 1.27 1.27) italic) hide)
     )
